File: PCB_v1/Payload_2026_PCB_v1.kicad_pcb (KiCad board)
At the start: 2 copper layers, 60 x 60 mm, 10 parts, among them J1 SD Card Reader, J2 Ozone Sensor, J3 SGP40 VOC Sensor, J4 IMU, J5 BME/BMP280, J6 Ultrasonic Sensor 1, J7 Ultrasonic Sensor 2, J8 Ultrasonic Sensor 3, J9 Battery

Commit message: Update PCB layout
Parts:
- moved J5 52.8 mm to (76.9, 30.1), turned to 0 degrees
- moved J9 20.7 mm to (31.4, 31.2), turned to 90 degrees
- moved J1 0.89 mm to (54.5, 33.0), turned to 180 degrees
Routing:
- net /GND: track 0.00 -> 17.3 mm
- net /SDA: track 54.3 -> 66.3 mm, vias 1 -> 0
- net /VIN: track 19.6 -> 9.58 mm
- net /SCL: track 67.1 -> 73.3 mm
- net /CLK / SCK: track 75.0 -> 71.5 mm
- net /DO / MISO: track 79.9 -> 76.9 mm
- net /CS: track 77.6 -> 79.6 mm
- net /DI / MOSI: track 78.8 -> 78.3 mm

Commit message: Update PCB Silkscreen Labels
Parts:
- J6: value Ultrasonic Sensor 1 -> Ultrasonic 1
- J7: value Ultrasonic Sensor 2 -> Ultrasonic 2
- J8: value Ultrasonic Sensor 3 -> Ultrasonic 3
Other:
- board text added: "5V"
- board text added: "Arduino Nano Every"
- board text added: "ECHO"
- board text added: "GND"
- board text added: "Payload 2026"
- board text added: "SCL"
- board text added: "SDA"
- board text added: "TRIG"
- board text added: "UA AIAA"
