File: PCB_v1/Payload_2026_PCB_v1.kicad_pcb (KiCad board)
At the start: 2 copper layers, 60 x 60 mm, 12 parts, among them J1 SD Card Reader, J10 SW-18020P, J2 Ozone Sensor, J3 SGP40 VOC Sensor, J4 IMU, J5 BME/BMP280, J6 Ultrasonic 1, J7 Ultrasonic 2, J8 Ultrasonic 3, J9 Battery

Commit message: Add another vibration sensor
Parts:
- removed ?: , clipboard:37f68170-0016-4afd-9e88-46bdadb5b772
- added J11: SW-18020P, Payload_2026_PCB_v1:SW_18020P, F.Cu at (42.0, 50.0)
Connections:
- net /SW_18020P renamed /SW_18020P_1
- A1 pad 26: unconnected-(A1-A7-Pad26) -> /SW_18020P_2
Routing:
- net /SW_18020P_2: track 0.00 -> 5.96 mm
